File: hardware/midi-solenoid-driver/midi-solenoid-driver.kicad_pcb (KiCad board)
At the start: 2 copper layers, 131.5 x 72 mm, 88 parts, among them J1 LEFT_DATA, J2 Conn_02x03_Odd_Even, J3 RIGHT_DATA, J4 12V_IN, J5 SOLENOIDS_OUT_1, J6 SOLENOIDS_OUT_2, Q1 Q_NMOS_GDS, Q10 Q_NMOS_GDS, Q11 Q_NMOS_GDS, Q12 Q_NMOS_GDS, Q13 Q_NMOS_GDS, Q14 Q_NMOS_GDS, Q15 Q_NMOS_GDS, Q16 Q_NMOS_GDS, Q2 Q_NMOS_GDS, Q3 Q_NMOS_GDS, Q4 Q_NMOS_GDS, Q5 Q_NMOS_GDS, Q6 Q_NMOS_GDS, Q7 Q_NMOS_GDS, Q8 Q_NMOS_GDS, Q9 Q_NMOS_GDS, SW1 MIDI_CHANNEl, SW2 SW_DIP_x08, U1 ATmega328PB-AU, U2 R-78B5.0-2.0, U3 SN75LBC176D

Commit message: Allow the pull-in to be PWM'd, not just the hold
The peak phase was the one time every energised channel drew full current at
once, and the only phase the per-channel stagger could not help. peakDutyPercent
now applies the same 500 Hz PWM and the same stagger to pull-in.

This matters most with solenoids overspecced for their load, which is the
common case. On 6.5 ohm 22 W units driving a small valve, 60% duty takes a
16-channel attack from 29.5 A to 10.2 A while still leaving roughly a 4:1
force margin over what the valve needs -- force falls as the square of coil
current, so the current drops far faster than the useful pull does.

At 100% the comparison against pwmPeriod constant-folds and the PWM branch is
optimised out entirely, so the default build is unchanged at 5726 bytes.

Bounds are enforced with static_assert: 0, 101 and negatives fail the build
rather than producing a solenoid that never seats. Also asserts pwmOnTime is
shorter than pwmPeriod.

README gains the worked example for a duty-cycle-limited solenoid, including
why bulk capacitance cannot cover a 40 ms attack, and how to read a "10% ED"
rating as a thermal budget when choosing hold duty.
Other:
- outline, holes or cut-outs redrawn
- net class Default removed
- net class FETs removed
